File: hardware/ml-ph-board.kicad_pcb (KiCad board)
At the start: 2 copper layers, 59.4 x 32.3 mm, 39 parts, among them J1 Conn_01x04_Male, J2 Conn_01x04, J3 BNCPTH, U1 ISO1540, U2 RFM-0505S, U3 STM8S003F3P, U4 LTC6081xMS8

Commit message: firmware
Parts:
- added C11: 0.1uF, Capacitor_SMD:C_0603_1608Metric, F.Cu at (136.9, 102.4)
- added R13: 1.5k, Resistor_SMD:R_0603_1608Metric, F.Cu at (136.9, 100.8)
- R6: value 1k -> 4.7k
- U4: footprint Package_SO:SO-8_5.3x6.2mm_P1.27mm -> Package_SO:SOIC-8_3.9x4.9mm_P1.27mm
- moved R9 1.52 mm to (136.9, 103.9)
Connections:
- J2 pad 1: /SWIM -> +5VD
- J2 pad 2: GNDD -> /SWIM
- J2 pad 3: +5VD -> GNDD
- U3 pad 3: Net-(U3-Pad3) -> /Aout
- U3 pad 5: /Aout -> Net-(R13-Pad1)
Routing:
- net +5VD: track 85.4 -> 94.6 mm
- net GNDD: track 21.1 -> 11.9 mm, vias 15 -> 16
- net (no net): track 48.2 -> 52.8 mm
- net Net-(R13-Pad1): track 0.00 -> 3.42 mm
- net Net-(C5-Pad1): track 9.40 -> 6.29 mm
- net Net-(R5-Pad2): track 11.3 -> 13.3 mm
- net /Aout: track 2.94 -> 4.57 mm
- net Net-(C11-Pad1): track 0.00 -> 1.53 mm
- net Net-(J3-PadS): track 4.95 -> 5.95 mm
- net Net-(C6-Pad1): track 31.9 -> 32.9 mm
- net /ADDR1: track 12.1 -> 11.2 mm
- net Net-(R6-Pad1): track 9.45 -> 10.3 mm
- net /SWIM: track 16.1 -> 15.3 mm
