File: hardware/ml-ph-board.kicad_pcb (KiCad board)
At the start: 2 copper layers, 59.4 x 32.3 mm, 41 parts, among them J1 Conn_01x04_Male, J2 Conn_01x04, J3 BNCPTH, U1 ISO1540, U2 RFM-0505S, U3 STM8S003F3P, U4 LTC6081xMS8

Commit message: Handle erroneous I2C signals
Other:
- board text added: "A0 Off On Off On"
- board text added: "A1 Off Off On On"
- board text added: "ADDR 0x45 0x44 0x43 0x42"
- board text removed: "A0 Off Off On On"
- board text removed: "A1 Off On Off On"
- board text removed: "ADDR 0x45 0x44 0x41 0x40"
Changed lines of the file:
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@@
     (34 B.Paste user)
     (35 F.Paste user)
-    (36 B.SilkS user hide)
+    (36 B.SilkS user)
     (37 F.SilkS user)
     (38 B.Mask user)
@@
     (solder_mask_min_width 0.25)
     (aux_axis_origin 0 0)
-    (visible_elements 7FFFFB7F)
+    (visible_elements 7FFFFFFF)
     (pcbplotparams
       (layerselection 0x010fc_ffffffff)
@@
   (gr_line (start 148.082 105.664) (end 148.082 115.57) (layer B.SilkS) (width 0.2))
   (gr_line (start 139.192 105.664) (end 148.082 105.664) (layer B.SilkS) (width 0.2))
-  (gr_text "ADDR\n0x45\n0x44\n0x41\n0x40" (at 143.764 113.538 90) (layer B.SilkS)
+  (gr_text "ADDR\n0x45\n0x44\n0x43\n0x42" (at 143.764 113.538 90) (layer B.SilkS)
     (effects (font (size 1 1) (thickness 0.15)) (justify mirror))
   )
-  (gr_text "A1\nOff\nOn\nOff\nOn" (at 143.764 109.728 90) (layer B.SilkS)
+  (gr_text "A0\nOff\nOn\nOff\nOn" (at 143.764 109.728 90) (layer B.SilkS)
     (effects (font (size 1 1) (thickness 0.15)) (justify mirror))
   )
-  (gr_text "A0\nOff\nOff\nOn\nOn" (at 143.764 107.188 90) (layer B.SilkS)
+  (gr_text "A1\nOff\nOff\nOn\nOn" (at 143.764 107.188 90) (layer B.SilkS)
     (effects (font (size 1 1) (thickness 0.15)) (justify mirror))
   )
@@
   (segment (start 131.385632 108.712) (end 131.385632 109.660368) (width 0.4) (layer F.Cu) (net 3))
   (segment (start 131.385632 109.660368) (end 130.556 110.49) (width 0.4) (layer F.Cu) (net 3))
-  (via (at 123.444 99.06) (size 0.8) (drill 0.4) (layers F.Cu B.Cu) (net 3))
+  (via (at 123.444 99.06) (size 0.8) (drill 0.4) (layers F.Cu B.Cu) (net 3) (status 1000000))
   (segment (start 122.809 99.695) (end 123.444 99.06) (width 0.4) (layer F.Cu) (net 3))
   (segment (start 123.444 99.06) (end 124.968 97.536) (width 0.4) (layer F.Cu) (net 3))
