File: hardware/ml-ph-board.sch (KiCad schematic (older format))
At the start: 38 parts, among them J1 Conn_01x04_Male, J2 Conn_01x04, J3 BNCPTH, U1 ISO1540, U2 RFM-0505S, U3 STM8S003F3P, U4 LTC6081xMS8

Commit message: firmware
Parts:
- added C11: 0.1uF, Capacitor_SMD:C_0603_1608Metric, symbol Device:C_Small
- added R13: 1.5k, Resistor_SMD:R_0603_1608Metric, symbol Device:R_Small_US
- R6: value 1k -> 4.7k
- U4: value LTC6081xMS8 -> LMC662xMS8; footprint Package_SO:SO-8_5.3x6.2mm_P1.27mm -> Package_SO:SOIC-8_3.9x4.9mm_P1.27mm
Connections:
- net +5VD: now also J2.1 (Pin_1); no longer J2.3 (Pin_3)
- net Aout: now also U3.3 (PD6), C11.2; no longer U3.5 (PA1)
- net GNDD: now also J2.3 (Pin_3); no longer J2.2 (Pin_2)
- net SWIM: now also J2.2 (Pin_2); no longer J2.1 (Pin_1)
- new net: R13.1, U3.5 (PA1)
- new net: C11.1, R13.2
- no-connect marks 9 -> 8
Changed lines of the file:
@@
 P 6700 1850
 F 0 "U4" H 6700 2217 50  0000 C CNN
-F 1 "LTC6081xMS8" H 6700 2126 50  0000 C CNN
-F 2 "Package_SO:SO-8_5.3x6.2mm_P1.27mm" H 6700 1850 50  0001 C CNN
+F 1 "LMC662xMS8" H 6700 2126 50  0000 C CNN
+F 2 "Package_SO:SOIC-8_3.9x4.9mm_P1.27mm" H 6700 1850 50  0001 C CNN
 F 3 "http://cds.linear.com/docs/en/datasheet/60812fd.pdf" H 6700 1850 50  0001 C CNN
 	1    6700 1850
@@
 P 6700 1850
 F 0 "U4" H 6658 1896 50  0000 L CNN
-F 1 "LTC6081xMS8" H 6658 1805 50  0000 L CNN
-F 2 "Package_SO:SO-8_5.3x6.2mm_P1.27mm" H 6700 1850 50  0001 C CNN
+F 1 "LMC662xMS8" H 6658 1805 50  0000 L CNN
+F 2 "Package_SO:SOIC-8_3.9x4.9mm_P1.27mm" H 6700 1850 50  0001 C CNN
 F 3 "http://cds.linear.com/docs/en/datasheet/60812fd.pdf" H 6700 1850 50  0001 C CNN
 	3    6700 1850
@@
 L power:+5VD #PWR0115
 U 1 1 5DF4A55D
-P 4250 5350
-F 0 "#PWR0115" H 4250 5200 50  0001 C CNN
-F 1 "+5VD" H 4265 5523 50  0000 C CNN
-F 2 "" H 4250 5350 50  0001 C CNN
-F 3 "" H 4250 5350 50  0001 C CNN
-	1    4250 5350
-	1    0    0    -1
+P 4150 5700
+F 0 "#PWR0115" H 4150 5550 50  0001 C CNN
+F 1 "+5VD" H 4165 5873 50  0000 C CNN
+F 2 "" H 4150 5700 50  0001 C CNN
+F 3 "" H 4150 5700 50  0001 C CNN
+	1    4150 5700
+	-1   0    0    1
 $EndComp
 $Comp
 L power:GNDD #PWR0116
 U 1 1 5DF4A586
-P 4250 5750
-F 0 "#PWR0116" H 4250 5500 50  0001 C CNN
-F 1 "GNDD" H 4254 5595 50  0000 C CNN
-F 2 "" H 4250 5750 50  0001 C CNN
-F 3 "" H 4250 5750 50  0001 C CNN
-	1    4250 5750
+P 4350 5550
+F 0 "#PWR0116" H 4350 5300 50  0001 C CNN
+F 1 "GNDD" H 4354 5395 50  0000 C CNN
+F 2 "" H 4350 5550 50  0001 C CNN
+F 3 "" H 4350 5550 50  0001 C CNN
+	1    4350 5550
 	1    0    0    -1
 $EndComp
 Wire Wire Line
 	3950 5400 4150 5400
-Text Label 4150 5700 2    50   ~ 0
+Text Label 4150 5600 2    50   ~ 0
 SWIM
 Wire Wire Line
@@
 P 8000 1550
 F 0 "R6" V 7795 1550 50  0000 C CNN
-F 1 "1k" V 7886 1550 50  0000 C CNN
+F 1 "4.7k" V 7886 1550 50  0000 C CNN
 F 2 "Resistor_SMD:R_0603_1608Metric" H 8000 1550 50  0001 C CNN
 F 3 "~" H 8000 1550 50  0001 C CNN
@@
 P 8050 1950
 F 0 "U4" H 8050 2317 50  0000 C CNN
-F 1 "LTC6081xMS8" H 8050 2226 50  0000 C CNN
-F 2 "Package_SO:SO-8_5.3x6.2mm_P1.27mm" H 8050 1950 50  0001 C CNN
+F 1 "LMC662xMS8" H 8050 2226 50  0000 C CNN
+F 2 "Package_SO:SOIC-8_3.9x4.9mm_P1.27mm" H 8050 1950 50  0001 C CNN
 F 3 "http://cds.linear.com/docs/en/datasheet/60812fd.pdf" H 8050 1950 50  0001 C CNN
 	2    8050 1950
@@
 	2550 1850 2550 1800
 Connection ~ 2550 1800
-Text Label 4900 3900 0    50   ~ 0
+Text Label 6650 4800 2    50   ~ 0
 Aout
 $Comp
@@
 NoConn ~ 5200 4600
 NoConn ~ 5200 4700
-NoConn ~ 5200 4800
 NoConn ~ 5200 4900
 NoConn ~ 5200 5000
 NoConn ~ 5200 4000
-NoConn ~ 6400 4800
 NoConn ~ 5200 4100
 Wire Wire Line
@@
 Text Label 6650 4700 2    50   ~ 0
 ADDR2
-Wire Wire Line
-	5200 3900 4900 3900
 $Comp
 L power:GNDD #PWR0124
@@
 	9250 1950 9000 1950
 Wire Wire Line
-	4250 5500 4250 5350
-Wire Wire Line
-	3950 5500 4250 5500
-Wire Wire Line
 	4250 5600 4250 5750
 Wire Wire Line
@@
 Text Notes 3050 1150 0    50   ~ 0
 RFM-0505S requires a minimum \ncurrent draw, so these resistors \nallow some wiggle room
+NoConn ~ 5200 4800
+Wire Wire Line
+	6400 4800 6650 4800
+$Comp
+L Device:R_Small_US R13
+U 1 1 5E0333DE
+P 5050 3900
+F 0 "R13" H 5118 3946 50  0000 L CNN
+F 1 "1.5k" H 5118 3855 50  0000 L CNN
+F 2 "Resistor_SMD:R_0603_1608Metric" H 5050 3900 50  0001 C CNN
+F 3 "~" H 5050 3900 50  0001 C CNN
+	1    5050 3900
+	0    1    1    0
+$EndComp
+$Comp
+L Device:C_Small C11
+U 1 1 5E033499
+P 4800 3900
+F 0 "C11" H 4892 3946 50  0000 L CNN
+F 1 "0.1uF" H 4892 3855 50  0000 L CNN
+F 2 "Capacitor_SMD:C_0603_1608Metric" H 4800 3900 50  0001 C CNN
+F 3 "~" H 4800 3900 50  0001 C CNN
+	1    4800 3900
+	0    1    1    0
+$EndComp
+Wire Wire Line
+	5150 3900 5200 3900
+Wire Wire Line
+	4950 3900 4900 3900
+Wire Wire Line
+	4700 3900 4500 3900
+Text Label 4500 3900 0    50   ~ 0
+Aout
+Wire Wire Line
+	4350 5500 4350 5550
+Wire Wire Line
+	3950 5500 4350 5500
 $EndSCHEMATC
